Commit message: Add HMMR sensor frames to Robot Desc

File: src/hmmr_description/urdf/hmmr.urdf.xacro (robot description, xacro)
@@ -48,3 +48,58 @@
         <origin xyz="0.25 0 0.30"/>
     </joint>
+    <!-- LiDAR Sensor -->
+    <link name="lidar_link">
+        <visual>
+            <geometry>
+                <cylinder radius="0.04" length="0.08"/>
+            </geometry>
+            <origin xyz="0 0 0"/>
+        </visual>
+    </link>
+    <joint name="lidar_joint" type="fixed">
+        <parent link="base_link"/>
+        <child link="lidar_link"/>
+        <origin xyz="0 0 0.32"/>
+    </joint>
+    <!-- IMU Sensor -->
+    <link name="imu_link">
+        <visual>
+            <geometry>
+                <box size="0.04 0.04 0.02"/>
+            </geometry>
+            <origin xyz="0 0 0"/>
+        </visual>
+    </link>
+    <joint name="imu_joint" type="fixed">
+        <parent link="base_link"/>
+        <child link="imu_link"/>
+        <origin xyz="0 0 0.15"/>
+    </joint>
+    <!-- Thermal Camera -->
+    <link name="thermal_camera_link">
+        <visual>
+            <geometry>
+                <box size="0.06 0.06 0.03"/>
+            </geometry>
+            <origin xyz="0 0 0"/>
+        </visual>
+    </link>
+    <joint name="thermal_camera_joint" type="fixed">
+        <parent link="base_link"/>
+        <child link="thermal_camera_link"/>
+        <origin xyz="-0.20 0 0.25"/>
+    </joint>
+    <!-- Environmental Sensor -->
+    <link name="environment_sensor_link">
+        <visual>
+            <geometry>
+                <sphere radius="0.03"/>
+            </geometry>
+        </visual>
+    </link>
+    <joint name="environment_sensor_joint" type="fixed">
+        <parent link="base_link"/>
+        <child link="environment_sensor_link"/>
+        <origin xyz="0 0.20 0.20"/>
+    </joint>
 </robot>
